File: Drum-K_MKII/Kicad/Controls.kicad_pcb (KiCad board)
At the start: 2 copper layers, 55.6 x 105.5 mm, 13 parts, among them J1 Conn_Left, J2 Conn_Right, J3 Accent, J4 Trig, J5 CV, J6 OUT, SW1 SW_Transient

Commit message: New Drum K
Changed lines of the file:
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@@
     (fp_rect (start -6.5 -4) (end 6.5 4)
       (stroke (width 0.1) (type default)) (fill none) (layer "F.Fab"))
-    (pad "1" thru_hole rect locked (at -4.699 0 90) (size 3 3) (drill oval 1.2 2.1) (layers "*.Cu" "*.Mask")
+    (pad "1" thru_hole rect locked (at -4.699 0 90) (size 3.3 3.5) (drill oval 1.5 2.5) (layers "*.Cu" "*.Mask")
       (net 1 "GND") (pinfunction "A") (pintype "passive"))
-    (pad "2" thru_hole circle locked (at 0 0 90) (size 3 3) (drill oval 1.2 2.1) (layers "*.Cu" "*.Mask")
+    (pad "2" thru_hole oval locked (at 0 0 90) (size 3.3 3.5) (drill oval 1.5 2.5) (layers "*.Cu" "*.Mask")
       (net 13 "SW1") (pinfunction "B") (pintype "passive"))
-    (pad "3" thru_hole circle locked (at 4.699 0 90) (size 3 3) (drill oval 1.2 2.1) (layers "*.Cu" "*.Mask"))
+    (pad "3" thru_hole oval locked (at 4.699 0 90) (size 3.3 3.5) (drill oval 1.5 2.5) (layers "*.Cu" "*.Mask"))
     (model "/home/plop/.local/share/kicad/7.0/3dmodels/Switchs/miniature-toggle-switches-mts-1xx-solder-terminal-1.snapshot.4/models3d/Toggle Switches/MTS-1xx-A1-blue.step"
       (offset (xyz 0 0 9.5))
