File: Drum-K_MKII/Kicad/Controls.kicad_sch (KiCad schematic)
At the start: 13 parts, among them J1 Conn_Left, J2 Conn_Right, J3 Accent, J4 Trig, J5 CV, J6 OUT, SW1 SW_Transient

Commit message: New Drum K
Parts:
- removed SW1: SW_Transient, Drum-K:Switch_MTS102, symbol Switch:SW_SPST
- added SW: SW_Transient, symbol Switch:SW_SPDT
Connections:
- net GND: now also SW.2 (B)
- net SW1: now also SW.1 (A)
- no-connect marks 0 -> 1
Changed lines of the file:
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@@
   (junction (at 36.83 55.88) (diameter 0) (color 0 0 0 0)
   )
+  (no_connect (at 110.49 123.19))
   (wire (pts (xy 114.3 50.8) (xy 118.11 50.8))
     (stroke (width 0) (type default))
@@
     )
   )
-  (global_label "SW1" (shape input) (at 110.49 125.73 180) (fields_autoplaced)
-    (effects (font (size 1.27 1.27)) (justify right))
-    (property "Intersheetrefs" "${INTERSHEET_REFS}" (at 103.7138 125.73 0)
+  (global_label "SW1" (shape input) (at 110.49 128.27 180) (fields_autoplaced)
+    (effects (font (size 1.27 1.27)) (justify right))
+    (property "Intersheetrefs" "${INTERSHEET_REFS}" (at 103.7138 128.27 0)
       (effects (font (size 1.27 1.27)) (justify right) hide)
     )
@@
     )
   )
+  (symbol (lib_id "Switch:SW_SPDT") (at 115.57 125.73 180) (unit 1)
+    (in_bom yes) (on_board yes) (dnp no)
+    (property "Reference" "SW" (at 115.57 118.11 0)
+      (effects (font (size 1.27 1.27)))
+    )
+    (property "Value" "SW_Transient" (at 115.57 120.65 0)
+      (effects (font (size 1.27 1.27)))
+    )
+    (property "Footprint" "" (at 115.57 125.73 0)
+      (effects (font (size 1.27 1.27)) hide)
+    )
+    (property "Datasheet" "~" (at 115.57 125.73 0)
+      (effects (font (size 1.27 1.27)) hide)
+    )
+    (pin "1")
+    (pin "2")
+    (pin "3")
+    (instances
+      (project "Controls"
+        (path "/363aee35-d89f-496c-8f19-1a4c6cfdf17b"
+          (reference "SW") (unit 1)
+        )
+      )
+    )
+  )
   (symbol (lib_id "power:GND") (at 118.11 91.44 0) (unit 1)
     (in_bom yes) (on_board yes) (dnp no) (fields_autoplaced)
@@
         )
       )
-    )
-  )
-  (symbol (lib_id "Switch:SW_SPST") (at 115.57 125.73 0) (mirror y) (unit 1)
-    (in_bom yes) (on_board yes) (dnp no)
-    (property "Reference" "SW1" (at 107.95 120.65 0)
-      (effects (font (size 1.27 1.27)))
-    )
-    (property "Value" "SW_Transient" (at 111.76 123.19 0)
-      (effects (font (size 1.27 1.27)))
-    )
-    (property "Footprint" "Drum-K:Switch_MTS102" (at 115.57 125.73 0)
-      (effects (font (size 1.27 1.27)) hide)
-    )
-    (property "Datasheet" "~" (at 115.57 125.73 0)
-      (effects (font (size 1.27 1.27)) hide)
-    )
-    (pin "1")
-    (pin "2")
-    (instances
-      (project "Controls"
-        (path "/363aee35-d89f-496c-8f19-1a4c6cfdf17b"
-          (reference "SW1") (unit 1)
-        )
-      )
-      (project "Drum-K_MKII"
-        (path "/580c517a-3259-445c-8dd8-1acd1cf1b729"
-          (reference "SW1") (unit 1)
-        )
-        (path "/580c517a-3259-445c-8dd8-1acd1cf1b729/d388ceb5-b2eb-4a81-900a-39560cadd23c"
-          (reference "SW2") (unit 1)
-        )
-      )
-      (project "Drum-kick"
-        (path "/e11a8019-98da-4172-96ca-3765cf26ae99"
-          (reference "SW1") (unit 1)
-        )
-      )
