File: Drum-K_MKII/Kicad/Drum-K_MKII.kicad_sch (KiCad schematic)
At the start: 90 parts, among them J1 Accent, J2 Trig, J3 Eurorack_power, J4 CV, J5 Conn_Left, J6 Conn_Right, J7 OUT, Q1 2N3904, Q2 2N3904, Q3 2N3906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

Commit message: New Drum K
Parts:
- removed SW1: SW_Transient, symbol Switch:SW_SPST
- added SW2: Transient, symbol Switch:SW_SPDT
Connections:
- net GND: now also SW2.1 (A)
- net SW1: now also SW2.2 (B)
- no-connect marks 0 -> 1
Changed lines of the file:
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@@
   (junction (at 104.14 248.92) (diameter 0) (color 0 0 0 0)
   )
-  (junction (at 209.55 39.37) (diameter 0) (color 0 0 0 0)
-  )
   (junction (at 207.01 66.04) (diameter 0) (color 0 0 0 0)
   )
@@
   (junction (at 156.21 72.39) (diameter 0) (color 0 0 0 0)
   )
+  (junction (at 209.55 39.37) (diameter 0) (color 0 0 0 0)
+  )
   (junction (at 148.59 229.87) (diameter 0) (color 0 0 0 0)
   )
@@
   (junction (at 165.1 72.39) (diameter 0) (color 0 0 0 0)
   )
+  (no_connect (at 199.39 36.83))
   (wire (pts (xy 375.92 142.24) (xy 377.19 142.24))
     (stroke (width 0) (type default))
@@
     (stroke (width 0) (type default))
   )
-  (wire (pts (xy 196.85 41.91) (xy 196.85 39.37))
+  (wire (pts (xy 196.85 44.45) (xy 196.85 41.91))
     (stroke (width 0) (type default))
   )
@@
     (stroke (width 0) (type default))
   )
+  (wire (pts (xy 209.55 39.37) (xy 209.55 44.45))
+    (stroke (width 0) (type default))
+  )
   (wire (pts (xy 137.16 243.84) (xy 128.27 243.84))
     (stroke (width 0) (type default))
@@
     (stroke (width 0) (type default))
   )
-  (wire (pts (xy 209.55 34.29) (xy 209.55 39.37))
-    (stroke (width 0) (type default))
-  )
   (wire (pts (xy 190.5 81.28) (xy 190.5 90.17))
     (stroke (width 0) (type default))
@@
     (stroke (width 0) (type default))
   )
-  (wire (pts (xy 209.55 39.37) (xy 209.55 44.45))
+  (wire (pts (xy 209.55 34.29) (xy 209.55 39.37))
     (stroke (width 0) (type default))
   )
@@
     (stroke (width 0) (type default))
   )
-  (wire (pts (xy 196.85 39.37) (xy 199.39 39.37))
+  (wire (pts (xy 196.85 41.91) (xy 199.39 41.91))
     (stroke (width 0) (type default))
   )
@@
     )
   )
+  (symbol (lib_id "Switch:SW_SPDT") (at 204.47 39.37 180) (unit 1)
+    (in_bom yes) (on_board yes) (dnp no) (fields_autoplaced)
+    (property "Reference" "SW2" (at 204.47 33.02 0)
+      (effects (font (size 1.27 1.27)))
+    )
+    (property "Value" "Transient" (at 204.47 35.56 0)
+      (effects (font (size 1.27 1.27)))
+    )
+    (property "Footprint" "" (at 204.47 39.37 0)
+      (effects (font (size 1.27 1.27)) hide)
+    )
+    (property "Datasheet" "~" (at 204.47 39.37 0)
+      (effects (font (size 1.27 1.27)) hide)
+    )
+    (pin "1")
+    (pin "2")
+    (pin "3")
+    (instances
+      (project "Drum-K_MKII"
+        (path "/580c517a-3259-445c-8dd8-1acd1cf1b729"
+          (reference "SW2") (unit 1)
+        )
+      )
+    )
+  )
   (symbol (lib_id "Device:R") (at 99.06 129.54 0) (unit 1)
     (in_bom yes) (on_board yes) (dnp no) (fields_autoplaced)
@@
     )
   )
-  (symbol (lib_id "Switch:SW_SPST") (at 204.47 39.37 0) (mirror y) (unit 1)
-    (in_bom yes) (on_board yes) (dnp no)
-    (property "Reference" "SW1" (at 196.85 34.29 0)
-      (effects (font (size 1.27 1.27)))
-    )
-    (property "Value" "SW_Transient" (at 200.66 36.83 0)
-      (effects (font (size 1.27 1.27)))
-    )
-    (property "Footprint" "" (at 204.47 39.37 0)
-      (effects (font (size 1.27 1.27)) hide)
-    )
-    (property "Datasheet" "~" (at 204.47 39.37 0)
-      (effects (font (size 1.27 1.27)) hide)
-    )
-    (pin "1")
-    (pin "2")
-    (instances
-      (project "Drum-K_MKII"
-        (path "/580c517a-3259-445c-8dd8-1acd1cf1b729"
-          (reference "SW1") (unit 1)
-        )
-      )
-      (project "Drum-kick"
-        (path "/e11a8019-98da-4172-96ca-3765cf26ae99"
-          (reference "SW1") (unit 1)
-        )
-      )
-    )
-  )
   (symbol (lib_id "Connector:TestPoint") (at 226.06 39.37 0) (unit 1)
     (in_bom yes) (on_board yes) (dnp no)
@@
     )
   )
-  (symbol (lib_id "power:GND") (at 196.85 41.91 0) (mirror y) (unit 1)
+  (symbol (lib_id "power:GND") (at 196.85 44.45 0) (mirror y) (unit 1)
     (in_bom yes) (on_board yes) (dnp no) (fields_autoplaced)
-    (property "Reference" "#PWR025" (at 196.85 48.26 0)
+    (property "Reference" "#PWR025" (at 196.85 50.8 0)
       (effects (font (size 1.27 1.27)) hide)
     )
-    (property "Value" "GND" (at 196.85 46.99 0)
+    (property "Value" "GND" (at 196.85 49.53 0)
       (effects (font (size 1.27 1.27)))
     )
-    (property "Footprint" "" (at 196.85 41.91 0)
+    (property "Footprint" "" (at 196.85 44.45 0)
       (effects (font (size 1.27 1.27)) hide)
     )
-    (property "Datasheet" "" (at 196.85 41.91 0)
+    (property "Datasheet" "" (at 196.85 44.45 0)
       (effects (font (size 1.27 1.27)) hide)
     )
